Commit message: Add MoveIt configuration and xarm_remote package with task server

File: src/xarm_description/urdf/xarm.xacro (robot description, xacro)
@@ -1,7 +1,11 @@
 <?xml version="1.0" ?>
 <robot name="xarm" xmlns:xacro="http://www.ros.org/wiki/xacro">
+<xacro:arg name="use_gazebo" default="false"/>
 <xacro:include filename="$(find xarm_description)/urdf/materials.xacro" />
 <xacro:include filename="$(find xarm_description)/urdf/xarm.gazebo" />
-<xacro:include filename="$(find xarm_description)/urdf/xarm.ros2_control.xacro" />
+<!-- Only include Gazebo ros2_control if use_gazebo is true -->
+<xacro:if value="$(arg use_gazebo)">
+  <xacro:include filename="$(find xarm_description)/urdf/xarm.ros2_control.xacro" />
+</xacro:if>
 <link name="base_link">
   <inertial>
@@ -188,5 +192,5 @@
     <origin xyz="-0.008709267199550398 0.0015004999553736196 0.023308296150939045" rpy="0 0 0"/>
     <mass value="0.012557670523597225"/>
-    <inertia ixx="3e-06" iyy="4e-06" izz="0.0" ixy="-0.0" iyz="0.0" ixz="1e-06"/>
+    <inertia ixx="3e-06" iyy="4e-06" izz="2e-06" ixy="-0.0" iyz="0.0" ixz="1e-06"/>
   </inertial>
   <visual>
@@ -208,5 +212,5 @@
     <origin xyz="0.008709194843970345 0.0015004999553735558 0.023308701233581364" rpy="0 0 0"/>
     <mass value="0.012557670523597225"/>
-    <inertia ixx="3e-06" iyy="4e-06" izz="0.0" ixy="0.0" iyz="0.0" ixz="-1e-06"/>
+    <inertia ixx="3e-06" iyy="4e-06" izz="2e-06" ixy="0.0" iyz="0.0" ixz="-1e-06"/>
   </inertial>
   <visual>
